File: LED_badge.kicad_pcb (KiCad board)
At the start: 2 copper layers, 60 x 60 mm, 19 parts, among them Q1 Q_NPN_CBE, SW1 SW_DPDT_x2

Commit message: update
Parts:
- added G***: LOGO, LED_badge:schematic, B.Cu at (134.9, 78.8)
- added G***: LOGO, LED_badge:robopotatoe, B.Cu at (156.0, 66.8)
- Q1: footprint Package_TO_SOT_THT:TO-92_Inline_Wide -> Package_TO_SOT_THT:TO-92_Inline
- moved SW1 2.00 mm to (134.5, 73.0)
- moved Q1 1.62 mm to (129.0, 66.3)
Routing:
- net Net-(D1-Pad1): track 10.9 -> 0.00 mm
- net Net-(R1-Pad1): track 9.88 -> 13.7 mm
- net Net-(BT1-Pad1): track 30.3 -> 28.3 mm
- net Net-(BT1-Pad2): track 46.7 -> 48.4 mm
- net Net-(Q1-Pad2): track 4.62 -> 5.62 mm
Other:
- net class Default: clearance 0.3 -> 0.2
- rule trace_clearance: 0.3 -> 0.2
- board text added: "ITF Fakultāte"
- board text added: "Un arī kartupeļbots, jo kapēc, gan ne"
- board text added: "Šeit ir shēma,ko šodien salodēji."
